Commit message: feat(AS-03): wire EZ-RASSOR meshes into the IPEx URDF visual (render-verified, not deferred)
The ROS/Gazebo rover now shows the articulated EZ-RASSOR meshes instead of primitive boxes/cylinders,
while KEEPING IPEx specs: per-link EZ-RASSOR glbs (rover_body/wheel/drum/drum_arm) baked to IPEx dims
(wheel dia 0.305, drum 0.437x0.353, chassis 0.46, arm reach 0.32) -> STL, wired into <visual>; <collision>
stays primitive (cylinder/box) for fast physics; inertials/joints/limits unchanged (still ipex_specs).
MIT attribution (THIRD_PARTY_LICENSES.txt) + measured transforms (MESH_TRANSFORMS.json). VERIFIED, not
container-gated: xacro expands + check_urdf parses the 18-child tree in stewie-ros2dev:jazzy, and the
assembled robot renders (yourdfpy+trimesh, xvfb) as a recognizable articulated RASSOR/IPEx rover -- image
pushed to gdrive Outbox. Guard: test_rig_contract.py [REQ:AS-03] (visual references the 4 meshes + assets
exist + collision stays primitive). rig contract 11/11, ruff clean.

File: ros2_ws/src/stewie_description/urdf/ipex.urdf.xacro (robot description, xacro)
@@ -56,5 +56,5 @@
       <visual>
         <origin rpy="${pi/2} 0 0"/>
-        <geometry><cylinder radius="${wheel_radius}" length="${wheel_width}"/></geometry>
+        <geometry><mesh filename="package://stewie_description/meshes/wheel.stl"/></geometry>
       </visual>
       <collision name="${name}_collision">
@@ -75,4 +75,7 @@
   <xacro:macro name="drum" params="name x">
     <link name="${name}_arm">
+      <visual>
+        <geometry><mesh filename="package://stewie_description/meshes/drum_arm.stl"/></geometry>
+      </visual>
       <xacro:box_inertial m="0.5" x="${drum_reach}" y="0.05" z="0.05"/>
     </link>
@@ -87,5 +90,5 @@
       <visual>
         <origin rpy="${pi/2} 0 0"/>
-        <geometry><cylinder radius="${drum_radius}" length="${drum_width}"/></geometry>
+        <geometry><mesh filename="package://stewie_description/meshes/drum.stl"/></geometry>
       </visual>
       <collision>
@@ -142,5 +145,5 @@
     <visual>
       <origin xyz="0 0 ${cg_height}"/>
-      <geometry><box size="${chassis_len} ${chassis_wid} ${chassis_hgt}"/></geometry>
+      <geometry><mesh filename="package://stewie_description/meshes/rover_body.stl"/></geometry>
     </visual>
     <collision>

Commit message: fix(AS-03): drum-arm joint continuous to match EZ-RASSOR articulation (cross-check)
Cross-checked STEWIE articulation against the EZ-RASSOR ROS2 URDF (FlaSpaceInst/ezrassor_sim_description):
wheel + drum-arm + drum-spin axes all 0 1 0 MATCH; EZ-RASSORs scale=0.35 mesh macro is exactly the
ROVER_SCALE=0.35 the sidecar referenced (educational size; STEWIE scales larger to IPEx specs). ONE real
difference: STEWIE pinned the drum arm to revolute +/-0.6 rad (an [ASSUMPTION]) while EZ-RASSOR uses a
CONTINUOUS arm -- RASSOR arms swing the drums dig<->dump, not a small lift. Changed STEWIEs drum_arm_joint
revolute -> continuous to match "all articulation like EZ-RASSOR", keeping effort = ARM_EXCAVATION_LOAD_NM
(18.5 Nm, IPEx spec). Verified: xacro expands, check_urdf parses, 8 continuous joints, rig contract 11/11.

File: ros2_ws/src/stewie_description/urdf/ipex.urdf.xacro (robot description, xacro)
@@ -80,10 +80,12 @@
       <xacro:box_inertial m="0.5" x="${drum_reach}" y="0.05" z="0.05"/>
     </link>
-    <joint name="${name}_arm_joint" type="revolute">
+    <joint name="${name}_arm_joint" type="continuous">
       <parent link="base_link"/>
       <child link="${name}_arm"/>
       <origin xyz="${x} 0 0"/>
       <axis xyz="0 1 0"/>
-      <limit lower="-0.6" upper="0.6" effort="${18.5}" velocity="1.0"/> <!-- ARM_EXCAVATION_LOAD_NM -->
+      <!-- continuous (full rotation) to match the EZ-RASSOR ROS2 URDF articulation: RASSOR arms swing
+           the drums dig<->dump, not a small revolute lift. effort = ARM_EXCAVATION_LOAD_NM (IPEx spec). -->
+      <limit effort="${18.5}" velocity="1.0"/>
     </joint>
     <link name="${name}">
