Commit message: feat(as+fs): land the concurrent AS-lane burst -- Gazebo seam, depth-source abstraction, FS-16 state routing
The AS-lane agent's (Codex) 3-hour-idle uncommitted burst, committed with four integration fixes
after a full local gate run (342+346 pytest across the touched lanes, 232/232 node --test, mypy
clean, ruff clean, req_trace reconciles, gen_status/manifest regenerated idempotently).

The burst: AS-02/03/05/06 verified-done (container-buildable ROS2 packages + IPEx description +
RViz dashboard + Gazebo seam, per-package import gates + rig contract tests); PM-13..16 rewritten
around a swappable depth-source abstraction (stereo/LiDAR/RGB-D/replay behind one DepthObservation
contract) + the cockpit design contract doc; FS-16 closed (cockpit_state.js loaded in production,
setView syncs through STEWIE_STATE, python gate test_cockpit_state_routing.py cites the row);
FS-15 X->D (Perception pane on normalizePerception); autonomy_contract topic-graph extensions;
release_gate + profiles depth-source validation; s3li crater writeup.

Integration fixes (would have redded CI): cockpit.js ?v= restamped (changed without a bump);
the 7 identical test/test_package_import.py collided in pytest ('test' package x7) -> unique
basenames + rootless dirs + a ros2_ws conftest path shim; stewie_msgs/FeatureTrackArray was
referenced by the frozen AS-01 topic contract but had no .msg -> FeatureTrack{,Array}.msg added
and registered; profiles.py shadowed a list-typed 'names' with a set (mypy).

File: ros2_ws/src/stewie_description/urdf/ipex.gazebo.xacro (robot description, xacro)
@@ -37,4 +37,17 @@
     </sensor>
   </gazebo>
+  <!-- Contact/collision evidence: front-left wheel contact sensor publishes when the rover settles
+       onto the regolith plane. gz sdf appends "_collision" to the named URDF collision, so the
+       sensor references the generated SDF collision name. It is diagnostics/evidence, not truth. -->
+  <gazebo reference="front_left_wheel">
+    <sensor name="front_left_wheel_contact" type="contact">
+      <always_on>1</always_on>
+      <update_rate>20</update_rate>
+      <contact>
+        <collision>front_left_wheel_collision_collision</collision>
+        <topic>/model/ipex/contact</topic>
+      </contact>
+    </sensor>
+  </gazebo>
   <!-- Front stereo cameras (RENDERING: needs the sensors system + a GL backend; GPU/EGL-gated headless).
        hfov 73.99 deg (profile optics), 1024x768; topics match the bridge camera entries. -->
@@ -63,3 +76,39 @@
     </sensor>
   </gazebo>
+  <!-- Selected simulated depth source for AS-06: low-rate front LiDAR-style cloud on the swappable
+       range-sensor mount. The no-LiDAR flight profile can still select stereo; this Gazebo source
+       gives the sim a concrete PointCloud2 egress without simulator truth. -->
+  <gazebo reference="lidar_front_mount">
+    <sensor name="lidar_front_points" type="gpu_lidar">
+      <always_on>1</always_on>
+      <update_rate>5</update_rate>
+      <topic>/model/ipex/perception</topic>
+      <lidar>
+        <scan>
+          <horizontal>
+            <samples>64</samples>
+            <resolution>1</resolution>
+            <min_angle>-0.785398</min_angle>
+            <max_angle>0.785398</max_angle>
+          </horizontal>
+          <vertical>
+            <samples>8</samples>
+            <resolution>1</resolution>
+            <min_angle>-0.261799</min_angle>
+            <max_angle>0.261799</max_angle>
+          </vertical>
+        </scan>
+        <range>
+          <min>0.20</min>
+          <max>20.0</max>
+          <resolution>0.02</resolution>
+        </range>
+        <noise>
+          <type>gaussian</type>
+          <mean>0.0</mean>
+          <stddev>0.01</stddev>
+        </noise>
+      </lidar>
+    </sensor>
+  </gazebo>
 </robot>

File: ros2_ws/src/stewie_description/urdf/ipex.urdf.xacro (robot description, xacro)
@@ -6,5 +6,5 @@
      via the `stereo_baseline` arg. The rejected 0.165 m shoulder split is documented in
      stewie/specs/stereo_authority.py and is deliberately NOT the default here.
-     Geometry provenance: stewie/specs/profile_data/stewie_ipex_v1.json (vehicle + stereo blocks)
+     Geometry provenance: stewie/specs/profile_data/stewie_ipex_v1.json (vehicle + stereo/sensor blocks)
      and stewie/specs/ipex_specs.py (SCHULER24 NTRS 20240008162 / WHEELTEST / BDSCALE). Per-part
      MASS ALLOCATION is [ASSUMPTION] (only the 30 kg dry total + 0.21 m CG height are sourced; the
@@ -58,5 +58,5 @@
         <geometry><cylinder radius="${wheel_radius}" length="${wheel_width}"/></geometry>
       </visual>
-      <collision>
+      <collision name="${name}_collision">
         <origin rpy="${pi/2} 0 0"/>
         <geometry><cylinder radius="${wheel_radius}" length="${wheel_width}"/></geometry>
@@ -123,4 +123,18 @@
     </joint>
   </xacro:macro>
+  <!-- Optional depth-source hardpoints. The selected source can be stereo, LiDAR, RGB-D, or replay;
+       the physical mount frames stay stable so downstream SLAM/mapping consumes the same cloud topic. -->
+  <xacro:macro name="depth_mount" params="name x y z yaw">
+    <link name="${name}">
+      <visual><geometry><box size="0.04 0.04 0.03"/></geometry></visual>
+      <collision><geometry><box size="0.04 0.04 0.03"/></geometry></collision>
+      <xacro:box_inertial m="0.08" x="0.04" y="0.04" z="0.03"/>
+    </link>
+    <joint name="${name}_joint" type="fixed">
+      <parent link="base_link"/>
+      <child link="${name}"/>
+      <origin xyz="${x} ${y} ${z}" rpy="0 0 ${yaw}"/>
+    </joint>
+  </xacro:macro>
   <!-- ============================ the robot ============================ -->
   <!-- base_link: the chassis body (REP-103 x-forward, y-left, z-up) -->
@@ -168,3 +182,8 @@
   <xacro:camera frame="drum_front"  x="${ wheelbase/2}" y="0" z="${cg_height}" yaw="0"/>
   <xacro:camera frame="drum_back"   x="${-wheelbase/2}" y="0" z="${cg_height}" yaw="${pi}"/>
+  <!-- Swappable depth-source mounts: stereo is flight-selected in the profile; LiDAR/RGB-D can be
+       installed on the same forward hardpoint when those sensors are available. -->
+  <xacro:depth_mount name="depth_sensor_mount" x="${ cam_fwd + 0.02}" y="0" z="${cam_z + 0.04}" yaw="0"/>
+  <xacro:depth_mount name="lidar_front_mount" x="${ cam_fwd + 0.03}" y="0" z="${cam_z + 0.07}" yaw="0"/>
+  <xacro:depth_mount name="rgbd_front_mount" x="${ cam_fwd + 0.03}" y="0" z="${cam_z + 0.04}" yaw="0"/>
 </robot>

Commit message: feat(BA-02): 8-camera rig with camera_info (glyph N->DDD)
The LAC-twin 8-camera rig now publishes image AND camera_info per camera, so perception can rectify/
triangulate. gazebo xacro: a gz_camera macro instantiates all 8 frames (front/rear stereo + L/R mono +
2 drum) each emitting <topic>/image + <camera_info_topic>/camera_info. autonomy_contract: CAMERA_FRAMES
+ 8 image + 8 CameraInfo topics. gz_bridge: 8 image + 8 camera_info bridged GZ_TO_ROS. Verified NOT
deferred: built stewie_description in stewie-ros2dev:jazzy and the gazebo overlay expands to 8 cameras +
8 camera_info_topics, check_urdf parses. Tests [REQ:BA-02] (every image has a paired camera_info in
contract + bridge) + BA-01 endpoint gate updated for the camera macro; ros2_ws suite green, mypy clean.

File: ros2_ws/src/stewie_description/urdf/ipex.gazebo.xacro (robot description, xacro)
@@ -50,30 +50,31 @@
     </sensor>
   </gazebo>
-  <!-- Front stereo cameras (RENDERING: needs the sensors system + a GL backend; GPU/EGL-gated headless).
-       hfov 73.99 deg (profile optics), 1024x768; topics match the bridge camera entries. -->
-  <gazebo reference="camera_front_left">
-    <sensor name="camera_front_left" type="camera">
-      <always_on>1</always_on>
-      <update_rate>10</update_rate>
-      <topic>/model/ipex/camera/front_left/image</topic>
-      <camera>
-        <horizontal_fov>1.2914</horizontal_fov>
-        <image><width>1024</width><height>768</height><format>R8G8B8</format></image>
-        <clip><near>0.02</near><far>100.0</far></clip>
-      </camera>
-    </sensor>
-  </gazebo>
-  <gazebo reference="camera_front_right">
-    <sensor name="camera_front_right" type="camera">
-      <always_on>1</always_on>
-      <update_rate>10</update_rate>
-      <topic>/model/ipex/camera/front_right/image</topic>
-      <camera>
-        <horizontal_fov>1.2914</horizontal_fov>
-        <image><width>1024</width><height>768</height><format>R8G8B8</format></image>
-        <clip><near>0.02</near><far>100.0</far></clip>
-      </camera>
-    </sensor>
-  </gazebo>
+  <!-- [BA-02] the LAC-twin 8-camera rig. Each camera emits its image AND its camera_info (intrinsics +
+       extrinsics) so perception can rectify/triangulate. hfov 73.99 deg (profile optics), 1024x768.
+       RENDERING needs the sensors system + a GL backend (GPU/EGL headless); the profile's max_live gates
+       which are active at runtime, but the description declares the full rig. -->
+  <xacro:macro name="gz_camera" params="frame">
+    <gazebo reference="camera_${frame}">
+      <sensor name="camera_${frame}" type="camera">
+        <always_on>1</always_on>
+        <update_rate>10</update_rate>
+        <topic>/model/ipex/camera/${frame}/image</topic>
+        <camera_info_topic>/model/ipex/camera/${frame}/camera_info</camera_info_topic>
+        <camera>
+          <horizontal_fov>1.2914</horizontal_fov>
+          <image><width>1024</width><height>768</height><format>R8G8B8</format></image>
+          <clip><near>0.02</near><far>100.0</far></clip>
+        </camera>
+      </sensor>
+    </gazebo>
+  </xacro:macro>
+  <xacro:gz_camera frame="front_left"/>
+  <xacro:gz_camera frame="front_right"/>
+  <xacro:gz_camera frame="rear_left"/>
+  <xacro:gz_camera frame="rear_right"/>
+  <xacro:gz_camera frame="left_mono"/>
+  <xacro:gz_camera frame="right_mono"/>
+  <xacro:gz_camera frame="drum_front"/>
+  <xacro:gz_camera frame="drum_back"/>
   <!-- Selected simulated depth source for AS-06: low-rate front LiDAR-style cloud on the swappable
        range-sensor mount. The no-LiDAR flight profile can still select stereo; this Gazebo source
